File: flight sim sch.sch (EAGLE design)
At the start: 87 parts, among them U1 MC74HC165ADGSOIC-16_ONS, U2 MC74HC165ADGSOIC-16_ONS, U3 MC74HC165ADGSOIC-16_ONS, U4 MC74HC165ADGSOIC-16_ONS, U5 MC74HC165ADGSOIC-16_ONS, U6 LMV324DR2GSOIC-14_NB_ONS-M, X1 332-16, X2 332-16, X3 332-16, X4 332-16, X5 332-16, X6 332-02, X7 332-02, X8 332-02, X9 332-02

Commit message: Add files via upload
Parts:
- renumbered 2C0.0033UF to C22, 2C0.003UF to C23, 2C0.47UF to C21, 2R27K to R213, 2R9.1K to R211, 2R91K to R212, 3C0.0033UF to C33, 3C0.22UF to C32, 3C0.47UF to C31, 3R27K to R313, 3R9.1K to R311, 3R91K to R312, 4C0.0033UF to C43, 4C0.22UF to C42, 4C0.47UF to C41, 4R27K to R413, 4R9.1K to R411, 4R91K to R412, C0.0033UF to C13, C0.22UF to C12, C0.47UF to C11, R27K to R113, R9.1K to R111, R91K to R112
Connections:
- removed net N$49: C100UF.-, SV1.3, SV2.3, SV3.3, SV4.3, U$1.GND, U1.CLOCKINHIBIT, U1.GND, U2.CLOCKINHIBIT, U2.GND, U3.CLOCKINHIBIT, U3.GND, U4.CLOCKINHIBIT, U4.GND, U5.CLOCKINHIBIT, U5.GND, U6.V-
- removed net N$67: C100UF.+, R1.2, R10.2, R11.2, R12.2, R13.2, R14.2, R15.2, R16.2, R17.2, R18.2, R19.2, R2.2, R20.2, R21.2, R22.2, R23.2, R24.2, R25.2, R26.2, R27.2, R28.2, R29.2, R3.2, R30.2, R31.2, R32.2, R33.2, R34.2, R35.2, R36.2, R37.2, R38.2, R39.2, R4.2, R40.2, R5.2, R6.2, R7.2, R8.2, R9.2, SV1.1, SV2.1, SV3.1, SV4.1, U$1.3.3V, U1.VCC, U2.VCC, U3.VCC, U4.VCC, U5.VCC, U6.V+
- new net 0: C100UF.-, C11.-, C13.-, C21.-, C23.-, C31.-, C33.-, C41.-, C43.-, SV1.3, SV2.3, SV3.3, SV4.3, U$1.GND, U1.CLOCKINHIBIT, U1.GND, U2.CLOCKINHIBIT, U2.GND, U3.CLOCKINHIBIT, U3.GND, U4.CLOCKINHIBIT, U4.GND, U5.CLOCKINHIBIT, U5.GND, U6.V-
- new net N$100: U3.VCC
- new net N$101: R33.2, R34.2, R35.2, R36.2, R37.2, R38.2, R39.2, R40.2
- new net N$102: U5.VCC
- new net N$103: C100UF.+, U$1.3.3V
- new net N$104: R17.2, R18.2, R19.2, R20.2, R21.2, R22.2, R23.2, R24.2
- new net N$105: R10.2, R11.2, R12.2, R13.2, R14.2, R15.2, R16.2, R9.2
- new net N$106: U2.VCC
- new net N$107: R1.2, R2.2, R3.2, R4.2, R5.2, R6.2, R7.2, R8.2
- new net N$108: U1.VCC
- net N$56: now also U6.V+; no longer C11.-, C13.-
- net N$59: now also SV1.1, SV2.1, SV3.1, SV4.1; no longer C21.-, C23.-
- net N$66: now also U4.VCC; no longer C31.-, C33.-
- net N$69: now also R25.2, R26.2, R27.2, R28.2, R29.2, R30.2, R31.2, R32.2; no longer C41.-, C43.-
Other:
- moved on the sheet: SV1, SV2, SV3, SV4

Commit message: Add files via upload
Parts:
- removed C100UF: (no value), rcl:CPOL-USE1.8-4
- removed X6, X7, X8, X9: 332-02, con-garry:332-02
- added C1: (no value), rcl:CPOL-USE1.8-4
- added SJ1, SJ2, SJ3, SJ4: (no value), jumper:SJ
Connections:
- net N$74 renamed N$B0
- net N$75 renamed N$B1
- net N$76 renamed N$B3
- net N$77 renamed N$B4
- net N$78 renamed N$B5
- net N$79 renamed N$B6
- net N$80 renamed N$B7
- net N$81 renamed N$B8
- net N$82 renamed N$B9
- net N$83 renamed N$B10
- net N$84 renamed N$B11
- net N$85 renamed N$B12
- net N$86 renamed N$B13
- net N$87 renamed N$B14
- net N$88 renamed N$B15
- net N$89 renamed N$A8
- net N$90 renamed N$A9
- net N$91 renamed N$A10
- net N$92 renamed N$A11
- net N$93 renamed N$A12
- net N$94 renamed N$A15
- net N$96 renamed N$C13
- net N$97 renamed N$C14
- net N$98 renamed N$C15
- removed net 0: C100UF.-, C11.-, C13.-, C21.-, C23.-, C31.-, C33.-, C41.-, C43.-, SV1.3, SV2.3, SV3.3, SV4.3, U$1.GND, U1.CLOCKINHIBIT, U1.GND, U2.CLOCKINHIBIT, U2.GND, U3.CLOCKINHIBIT, U3.GND, U4.CLOCKINHIBIT, U4.GND, U5.CLOCKINHIBIT, U5.GND, U6.V-
- removed net N$100: U3.VCC
- removed net N$101: R33.2, R34.2, R35.2, R36.2, R37.2, R38.2, R39.2, R40.2
- removed net N$102: U5.VCC
- removed net N$103: C100UF.+, U$1.3.3V
- removed net N$104: R17.2, R18.2, R19.2, R20.2, R21.2, R22.2, R23.2, R24.2
- removed net N$105: R10.2, R11.2, R12.2, R13.2, R14.2, R15.2, R16.2, R9.2
- removed net N$106: U2.VCC
- removed net N$107: R1.2, R2.2, R3.2, R4.2, R5.2, R6.2, R7.2, R8.2
- removed net N$108: U1.VCC
- removed net N$12: R14.1, U2.G
- removed net N$17: R9.1, U2.D
- removed net N$43: U$1.PA_3, U1.CLOCK, U2.CLOCK, U3.CLOCK, U4.CLOCK, U5.CLOCK
- removed net N$59: SV1.1, SV2.1, SV3.1, SV4.1
- removed net N$61: R211.2, SV2.2
- removed net N$63: R311.1, SV3.2
- removed net N$66: U4.VCC
- removed net N$69: R25.2, R26.2, R27.2, R28.2, R29.2, R30.2, R31.2, R32.2
- removed net N$70: C42.+, R412.2, R413.1, U$1.PA_1, X8-1.S
- removed net N$71: C12.-, U6.INA-, U6.OUTA
- removed net N$73: C22.-, U6.INB-, U6.OUTB
- new net AGND: C1.-, C11.-, C13.-, C21.-, C23.-, C31.-, C33.-, C41.-, C43.-, U$1.GND, U1.CLOCKINHIBIT, U1.GND, U2.CLOCKINHIBIT, U2.GND, U3.CLOCKINHIBIT, U3.GND, U4.CLOCKINHIBIT, U4.GND, U5.CLOCKINHIBIT, U5.GND, U6.V+, U6.V-
- new net DGND: SV1.3, SV2.3, SV3.3, SV4.3
- new net N$49: R40.2, U5.H
- new net N$FILTER2OUT: C22.+, SJ2.1, U$1.PA_6, U6.INB-, U6.OUTB
- new net N$FILTER3OUT: C32.+, SJ3.1, U$1.PA_0, U6.IND-, U6.OUTD
- new net N$FILTER4OUT: C42.+, SJ4.1, U$1.PA_1, U6.INC-, U6.OUTC
- new net N$POT1IN: R111.2, SJ1.2, SV1.2
- new net N$POT2IN: R211.2, SJ2.2, SV2.2
- new net N$POT3IN: R311.1, SJ3.2, SV3.2
- new net N$POT4IN: R411.1, SJ4.2, SV4.2
- new net VCC: C1.+, R1.1, R10.1, R11.1, R12.1, R13.1, R14.1, R15.1, R16.1, R17.1, R18.1, R19.1, R2.1, R20.1, R21.1, R22.1, R23.1, R24.1, R25.1, R26.1, R27.1, R28.1, R29.1, R3.1, R30.1, R31.1, R32.1, R33.1, R34.1, R35.1, R36.1, R37.1, R38.1, R39.1, R4.1, R40.1, R5.1, R6.1, R7.1, R8.1, R9.1, SV1.1, SV2.1, SV3.1, SV4.1, U$1.3.3V, U1.VCC, U2.VCC, U3.VCC, U4.VCC, U5.VCC
- net N$10: now also U$1.PA_3, U2.CLOCK, U3.CLOCK, U4.CLOCK, U5.CLOCK; no longer R16.1, U2.E
- net N$11: now also U1.CLOCK; no longer R15.1, U2.F
- net N$13: now also R16.2; no longer R13.1
- net N$14: now also R15.2, U2.G; no longer R12.1, U2.A
- net N$15: now also R14.2, U2.F; no longer R11.1, U2.B
- net N$16: now also R13.2, U2.E; no longer R10.1, U2.C
- net N$18: now also R24.2, U3.H; no longer R24.1, U3.E
- net N$19: now also R23.2, U3.G; no longer R23.1, U3.F
- net N$2: now also R8.2, U1.H; no longer R8.1, U1.E
- net N$20: now also R22.2, U3.F; no longer R22.1, U3.G
- net N$21: now also R21.2, U3.E; no longer R21.1, U3.H
- net N$22: now also R20.2, U3.D; no longer R20.1, U3.A
- net N$23: now also R19.2, U3.C; no longer R19.1, U3.B
- net N$24: now also R18.2, U3.B; no longer R18.1, U3.C
- net N$25: now also R12.2, U2.D; no longer R17.1, U3.D
- net N$26: now also R32.2, U4.H; no longer R32.1, U4.E
- net N$27: now also R31.2, U4.G; no longer R31.1, U4.F
- net N$28: now also R30.2, U4.F; no longer R30.1, U4.G
- net N$29: now also R29.2, U4.E; no longer R29.1, U4.H
- net N$3: now also R7.2, U1.G; no longer R7.1, U1.F
- net N$30: now also R28.2, U4.D; no longer R28.1, U4.A
- net N$31: now also R27.2, U4.C; no longer R27.1, U4.B
- net N$32: now also R26.2, U4.B; no longer R26.1, U4.C
- net N$33: now also R33.2, U5.A; no longer R40.1, U5.E
- net N$34: now also R25.2, U4.A; no longer R39.1, U5.F
- net N$35: now also R34.2, U5.B; no longer R38.1, U5.G
- net N$36: now also R11.2, U2.C; no longer R25.1, U4.D
- net N$37: now also R35.2, U5.C; no longer R37.1, U5.H
- net N$38: now also R36.2, U5.D; no longer R36.1, U5.A
- net N$39: now also R37.2, U5.E; no longer R35.1, U5.B
- net N$4: now also R6.2, U1.F; no longer R6.1, U1.G
- net N$40: now also R38.2, U5.F; no longer R34.1, U5.C
- net N$41: now also R39.2, U5.G; no longer R33.1, U5.D
- net N$5: now also R5.2, U1.E; no longer R5.1, U1.H
- net N$50: now also C22.-, R212.1, R213.2; no longer C12.+, R112.1, R113.2, U$1.PA_7, X9-1.S
- net N$53: now also C12.+, SJ1.1, U$1.PA_7, U6.INA-, U6.OUTA; no longer C42.-, U6.INC-, U6.OUTC
- net N$54: now also C12.-, R112.1, R113.2; no longer R411.1, SV4.2
- net N$55: now also R10.2, U2.B; no longer C32.-, U$1.PA_0, U6.IND-, U6.OUTD, X7-1.S
- net N$56: now also R9.2, U2.A; no longer U6.V+
- net N$57: now also C42.-, R412.2, R413.1; no longer C22.+, R212.1, R213.2, U$1.PA_6, X6-1.S
- net N$6: now also R4.2, U1.D; no longer R4.1, U1.A
- net N$60: now also R17.2, U3.A; no longer R111.2, SV1.2
- net N$7: now also R3.2, U1.C; no longer R3.1, U1.B
- net N$72: now also C32.-; no longer C32.+
- net N$8: now also R2.2, U1.B; no longer R2.1, U1.C
- net N$9: now also R1.2, U1.A; no longer R1.1, U1.D
Other:
- moved on the sheet: C12, C22, C31, C32, C33, C42, R1, R10, R11, R12, R13, R14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

Commit message: Add files via upload
Connections:
- net AGND: now also X1-1.S, X1-11.S, X1-13.S, X1-15.S, X1-3.S, X1-5.S, X1-7.S, X1-9.S, X2-1.S, X2-11.S, X2-13.S, X2-15.S, X2-3.S, X2-5.S, X2-7.S, X2-9.S, X3-1.S, X3-11.S, X3-13.S, X3-15.S, X3-3.S, X3-5.S, X3-7.S, X3-9.S, X4-1.S, X4-11.S, X4-13.S, X4-15.S, X4-3.S, X4-5.S, X4-7.S, X4-9.S, X5-1.S, X5-11.S, X5-13.S, X5-15.S, X5-3.S, X5-5.S, X5-7.S, X5-9.S
- net N$13: now also X2-16.S
- net N$14: now also X2-14.S
- net N$15: now also X2-12.S
- net N$16: now also X2-10.S
- net N$18: now also X3-16.S
- net N$19: now also X3-14.S
- net N$2: now also X1-16.S
- net N$20: now also X3-12.S
- net N$21: now also X3-10.S
- net N$22: now also X3-8.S
- net N$23: now also X3-6.S
- net N$24: now also X3-4.S
- net N$25: now also X2-8.S
- net N$26: now also X4-16.S
- net N$27: now also X4-14.S
- net N$28: now also X4-12.S
- net N$29: now also X4-10.S
- net N$3: now also X1-14.S
- net N$30: now also X4-8.S
- net N$31: now also X4-6.S
- net N$32: now also X4-4.S
- net N$33: now also X5-2.S
- net N$34: now also X4-2.S
- net N$35: now also X5-4.S
- net N$36: now also X2-6.S
- net N$37: now also X5-6.S
- net N$38: now also X5-8.S
- net N$39: now also X5-10.S
- net N$4: now also X1-12.S
- net N$40: now also X5-12.S
- net N$41: now also X5-14.S
- net N$49: now also X5-16.S
- net N$5: now also X1-10.S
- net N$55: now also X2-4.S
- net N$56: now also X2-2.S
- net N$6: now also X1-8.S
- net N$60: now also X3-2.S
- net N$7: now also X1-6.S
- net N$8: now also X1-4.S
- net N$9: now also X1-2.S
Other:
- moved on the sheet: X1-1, X1-10, X1-11, X1-12, X1-13, X1-14, X1-15, X1-16, X1-2, X1-3, X1-4, X1-5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

Commit message: Add files via upload
Parts:
- removed X1, X2, X3, X4, X5: 332-16, con-garry:332-16
- added SV10, SV11, SV7, SV8, SV9: (no value), con-lstb:MA08-2
Connections:
- removed net N$11: U1.CLOCK
- net AGND: now also SV10.10, SV10.12, SV10.14, SV10.16, SV10.2, SV10.4, SV10.6, SV10.8, SV11.10, SV11.12, SV11.14, SV11.16, SV11.2, SV11.4, SV11.6, SV11.8, SV7.10, SV7.12, SV7.14, SV7.16, SV7.2, SV7.4, SV7.6, SV7.8, SV8.10, SV8.12, SV8.14, SV8.16, SV8.2, SV8.4, SV8.6, SV8.8, SV9.10, SV9.12, SV9.14, SV9.16, SV9.2, SV9.4, SV9.6, SV9.8; no longer X1-1.S, X1-11.S, X1-13.S, X1-15.S, X1-3.S, X1-5.S, X1-7.S, X1-9.S, X2-1.S, X2-11.S, X2-13.S, X2-15.S, X2-3.S, X2-5.S, X2-7.S, X2-9.S, X3-1.S, X3-11.S, X3-13.S, X3-15.S, X3-3.S, X3-5.S, X3-7.S, X3-9.S, X4-1.S, X4-11.S, X4-13.S, X4-15.S, X4-3.S, X4-5.S, X4-7.S, X4-9.S, X5-1.S, X5-11.S, X5-13.S, X5-15.S, X5-3.S, X5-5.S, X5-7.S, X5-9.S
- net N$10: now also U1.CLOCK
- net N$13: now also SV8.1; no longer X2-16.S
- net N$14: now also SV8.3; no longer X2-14.S
- net N$15: now also SV8.5; no longer X2-12.S
- net N$16: now also SV8.7; no longer X2-10.S
- net N$18: now also SV9.1; no longer X3-16.S
- net N$19: now also SV9.3; no longer X3-14.S
- net N$2: now also SV7.1; no longer X1-16.S
- net N$20: now also SV9.5; no longer X3-12.S
- net N$21: now also SV9.7; no longer X3-10.S
- net N$22: now also SV9.9; no longer X3-8.S
- net N$23: now also SV9.11; no longer X3-6.S
- net N$24: now also SV9.13; no longer X3-4.S
- net N$25: now also SV8.9; no longer X2-8.S
- net N$26: now also SV10.1; no longer X4-16.S
- net N$27: now also SV10.3; no longer X4-14.S
- net N$28: now also SV10.5; no longer X4-12.S
- net N$29: now also SV10.7; no longer X4-10.S
- net N$3: now also SV7.3; no longer X1-14.S
- net N$30: now also SV10.9; no longer X4-8.S
- net N$31: now also SV10.11; no longer X4-6.S
- net N$32: now also SV10.13; no longer X4-4.S
- net N$33: now also SV11.15; no longer X5-2.S
- net N$34: now also SV10.15; no longer X4-2.S
- net N$35: now also SV11.13; no longer X5-4.S
- net N$36: now also SV8.11; no longer X2-6.S
- net N$37: now also SV11.11; no longer X5-6.S
- net N$38: now also SV11.9; no longer X5-8.S
- net N$39: now also SV11.7; no longer X5-10.S
- net N$4: now also SV7.5; no longer X1-12.S
- net N$40: now also SV11.5; no longer X5-12.S
- net N$41: now also SV11.3; no longer X5-14.S
- net N$49: now also SV11.1; no longer X5-16.S
- net N$5: now also SV7.7; no longer X1-10.S
- net N$55: now also SV8.13; no longer X2-4.S
- net N$56: now also SV8.15; no longer X2-2.S
- net N$6: now also SV7.9; no longer X1-8.S
- net N$60: now also SV9.15; no longer X3-2.S
- net N$7: now also SV7.11; no longer X1-6.S
- net N$8: now also SV7.13; no longer X1-4.S
- net N$9: now also SV7.15; no longer X1-2.S
Other:
- moved on the sheet: R25, R26, R27, R28, R29, R30, R31, R32, R33, R34, R35, R36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

Commit message: Add files via upload
Connections:
- net AGND: no longer U6.V+
- net VCC: now also U6.V+
Changed lines of the file:
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@@
 <part name="SJ3" library="jumper" library_urn="urn:adsk.eagle:library:252" deviceset="SJ" device="" package3d_urn="urn:adsk.eagle:package:15471/1"/>
 <part name="SJ4" library="jumper" library_urn="urn:adsk.eagle:library:252" deviceset="SJ" device="" package3d_urn="urn:adsk.eagle:package:15471/1"/>
-<part name="SUPPLY15" library="supply2" library_urn="urn:adsk.eagle:library:372" deviceset="AGND" device=""/>
 <part name="SUPPLY16" library="supply2" library_urn="urn:adsk.eagle:library:372" deviceset="AGND" device=""/>
 <part name="SUPPLY17" library="supply2" library_urn="urn:adsk.eagle:library:372" deviceset="AGND" device=""/>
@@
 <part name="SV10" library="con-lstb" library_urn="urn:adsk.eagle:library:162" deviceset="MA08-2" device="" package3d_urn="urn:adsk.eagle:package:8335/1"/>
 <part name="SV11" library="con-lstb" library_urn="urn:adsk.eagle:library:162" deviceset="MA08-2" device="" package3d_urn="urn:adsk.eagle:package:8335/1"/>
+<part name="P+4" library="supply1" library_urn="urn:adsk.eagle:library:371" deviceset="VCC" device=""/>
 </parts>
 <sheets>
@@
 <attribute name="VALUE" x="431.8" y="46.99" size="1.778" layer="96"/>
 </instance>
-<instance part="SUPPLY15" gate="G$1" x="416.56" y="-2.54" smashed="yes" rot="R270">
-<attribute name="VALUE" x="413.385" y="0.127" size="1.778" layer="96" rot="R270"/>
-</instance>
 <instance part="SUPPLY16" gate="G$1" x="-2.54" y="35.56" smashed="yes">
 <attribute name="VALUE" x="-5.207" y="32.385" size="1.778" layer="96"/>
@@
 <attribute name="VALUE" x="-49.53" y="-114.3" size="1.778" layer="96"/>
 <attribute name="NAME" x="-49.53" y="-88.138" size="1.778" layer="95"/>
+</instance>
+<instance part="P+4" gate="VCC" x="416.56" y="-2.54" smashed="yes" rot="R90">
+<attribute name="VALUE" x="419.1" y="-5.08" size="1.778" layer="96" rot="R180"/>
 </instance>
 </instances>
@@
 <pinref part="P+3" gate="VCC" pin="VCC"/>
 </segment>
+<segment>
+<pinref part="U6" gate="A" pin="V+"/>
+<wire x1="421.64" y1="-2.54" x2="419.1" y2="-2.54" width="0.1524" layer="91"/>
+<pinref part="P+4" gate="VCC" pin="VCC"/>
+</segment>
 </net>
 <net name="N$54" class="0">
@@
 <junction x="414.02" y="58.42"/>
 <pinref part="SJ3" gate="1" pin="1"/>
+<junction x="459.74" y="20.32"/>
 </segment>
 </net>
@@
 <wire x1="391.16" y1="-7.62" x2="391.16" y2="-5.08" width="0.1524" layer="91"/>
 <pinref part="SUPPLY6" gate="G$1" pin="AGND"/>
+<junction x="391.16" y="-5.08"/>
 </segment>
 <segment>
@@
 </segment>
 <segment>
-<pinref part="U6" gate="A" pin="V+"/>
-<wire x1="421.64" y1="-2.54" x2="419.1" y2="-2.54" width="0.1524" layer="91"/>
-<pinref part="SUPPLY15" gate="G$1" pin="AGND"/>
-</segment>
-<segment>
