File: flight sim sch.brd (EAGLE design)
At the start: 255.2 x 103.8 mm, 87 parts, among them U1 MC74HC165ADGSOIC-16_ONS, U2 MC74HC165ADGSOIC-16_ONS, U3 MC74HC165ADGSOIC-16_ONS, U4 MC74HC165ADGSOIC-16_ONS, U5 MC74HC165ADGSOIC-16_ONS, U6 LMV324DR2GSOIC-14_NB_ONS-M, X1 332-16, X2 332-16, X3 332-16, X4 332-16, X5 332-16

Commit message: trial layout ideas
Parts:
- moved U2 83.5 mm to (46.4, 76.8), turned to 270 degrees
- moved U1 80.8 mm to (24.1, 76.2)
- moved R9 50.2 mm to (40.6, 95.9), turned to 270 degrees
- moved R1 49.8 mm to (33.0, 83.8), turned to 90 degrees
- moved R10 44.3 mm to (45.7, 95.9), turned to 270 degrees
- moved R2 43.3 mm to (30.5, 83.8), turned to 90 degrees
- moved U$1 40.7 mm to (43.2, 58.4)
- moved R17 39.4 mm to (78.7, 83.8), turned to 90 degrees
- moved R11 39.2 mm to (50.8, 95.9), turned to 270 degrees
- moved SV6 39.2 mm to (21.0, 40.0), turned to 180 degrees
- moved SV5 38.8 mm to (62.9, 40.0)
- moved R3 36.8 mm to (27.9, 83.8), turned to 90 degrees
- moved R12 35.2 mm to (55.9, 95.9), turned to 270 degrees
- moved R18 33.1 mm to (76.2, 83.8), turned to 90 degrees
- moved R4 30.6 mm to (25.4, 83.8), turned to 90 degrees
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Routing:
- net N$9: track 0.00 -> 28.8 mm
- net N$2: track 0.00 -> 25.5 mm
- net N$8: track 0.00 -> 25.0 mm
- net N$3: track 0.00 -> 22.1 mm
- net N$4: track 0.00 -> 21.7 mm
- net N$7: track 0.00 -> 21.2 mm
- net N$6: track 0.00 -> 20.8 mm
- net N$5: track 0.00 -> 20.3 mm
- net N$25: track 0.00 -> 16.6 mm
- net N$56: track 0.00 -> 14.0 mm
- net N$36: track 0.00 -> 12.4 mm
- net N$55: track 0.00 -> 10.6 mm
- net N$13: track 0.00 -> 10.3 mm
- net N$16: track 0.00 -> 8.88 mm
- net N$14: track 0.00 -> 6.08 mm
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
Commit message: Add files via upload
Parts:
- removed X1, X2, X3, X4, X5: 332-16, con-garry:332-16
- added SV10, SV11, SV7, SV8, SV9: (no value), con-lstb:MA08-2
- moved SV1 166.3 mm to (82.5, 3.81), turned to 180 degrees
- moved SV2 151.6 mm to (100.3, 3.81), turned to 180 degrees
- moved C12 147.7 mm to (78.7, 15.2)
- moved SJ1 141.1 mm to (86.4, 19.1)
- moved R112 139.7 mm to (76.2, 7.62), turned to 0 degrees
- moved SV3 138.7 mm to (118.1, 3.81), turned to 180 degrees
- moved R113 133.6 mm to (87.6, 11.4), turned to 180 degrees
- moved SV4 128.7 mm to (137.2, 3.81), turned to 180 degrees
- moved R212 127.4 mm to (95.2, 7.62), turned to 0 degrees
- moved C13 125.6 mm to (90.2, 3.81)
- moved C21 122.5 mm to (109.2, 3.81), turned to 180 degrees
- moved C11 119.4 mm to (85.1, 15.2), turned to 0 degrees
- moved R211 117.3 mm to (109.2, 7.62), turned to 90 degrees
- moved C22 117.1 mm to (96.5, 15.2), turned to 180 degrees
- moved C41 114.9 mm to (144.8, 3.81), turned to 180 degrees
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Connections:
- removed net N$11: U1.2
- net AGND: now also SV10.10, SV10.12, SV10.14, SV10.16, SV10.2, SV10.4, SV10.6, SV10.8, SV11.10, SV11.12, SV11.14, SV11.16, SV11.2, SV11.4, SV11.6, SV11.8, SV7.10, SV7.12, SV7.14, SV7.16, SV7.2, SV7.4, SV7.6, SV7.8, SV8.10, SV8.12, SV8.14, SV8.16, SV8.2, SV8.4, SV8.6, SV8.8, SV9.10, SV9.12, SV9.14, SV9.16, SV9.2, SV9.4, SV9.6, SV9.8; no longer X1.1, X1.11, X1.13, X1.15, X1.3, X1.5, X1.7, X1.9, X2.1, X2.11, X2.13, X2.15, X2.3, X2.5, X2.7, X2.9, X3.1, X3.11, X3.13, X3.15, X3.3, X3.5, X3.7, X3.9, X4.1, X4.11, X4.13, X4.15, X4.3, X4.5, X4.7, X4.9, X5.1, X5.11, X5.13, X5.15, X5.3, X5.5, X5.7, X5.9
- net N$10: now also U1.2
- net N$13: now also SV8.1; no longer X2.16
- net N$14: now also SV8.3; no longer X2.14
- net N$15: now also SV8.5; no longer X2.12
- net N$16: now also SV8.7; no longer X2.10
- net N$18: now also SV9.1; no longer X3.16
- net N$19: now also SV9.3; no longer X3.14
- net N$2: now also SV7.1; no longer X1.16
- net N$20: now also SV9.5; no longer X3.12
- net N$21: now also SV9.7; no longer X3.10
- net N$22: now also SV9.9; no longer X3.8
- net N$23: now also SV9.11; no longer X3.6
- net N$24: now also SV9.13; no longer X3.4
- net N$25: now also SV8.9; no longer X2.8
- net N$26: now also SV10.1; no longer X4.16
- net N$27: now also SV10.3; no longer X4.14
- net N$28: now also SV10.5; no longer X4.12
- net N$29: now also SV10.7; no longer X4.10
- net N$3: now also SV7.3; no longer X1.14
- net N$30: now also SV10.9; no longer X4.8
- net N$31: now also SV10.11; no longer X4.6
- net N$32: now also SV10.13; no longer X4.4
- net N$33: now also SV11.15; no longer X5.2
- net N$34: now also SV10.15; no longer X4.2
- net N$35: now also SV11.13; no longer X5.4
- net N$36: now also SV8.11; no longer X2.6
- net N$37: now also SV11.11; no longer X5.6
- net N$38: now also SV11.9; no longer X5.8
- net N$39: now also SV11.7; no longer X5.10
- net N$4: now also SV7.5; no longer X1.12
- net N$40: now also SV11.5; no longer X5.12
- net N$41: now also SV11.3; no longer X5.14
- net N$49: now also SV11.1; no longer X5.16
- net N$5: now also SV7.7; no longer X1.10
- net N$55: now also SV8.13; no longer X2.4
- net N$56: now also SV8.15; no longer X2.2
- net N$6: now also SV7.9; no longer X1.8
- net N$60: now also SV9.15; no longer X3.2
- net N$7: now also SV7.11; no longer X1.6
- net N$8: now also SV7.13; no longer X1.4
- net N$9: now also SV7.15; no longer X1.2
Routing:
- net AGND: track 0.00 -> 556.8 mm, vias 0 -> 2
- net VCC: track 0.00 -> 356.2 mm, vias 0 -> 5
- net N$47: track 0.00 -> 175.7 mm, vias 0 -> 1
- net N$48: track 0.00 -> 167.5 mm, vias 0 -> 5
- net N$10: track 0.00 -> 167.1 mm, vias 0 -> 5
- net N$FILTER4OUT: track 0.00 -> 107.3 mm, vias 0 -> 1
- net N$FILTER3OUT: track 0.00 -> 101.5 mm, vias 0 -> 3
- net N$53: track 0.00 -> 96.0 mm
- net N$FILTER2OUT: track 0.00 -> 93.6 mm
- net N$B12: track 0.00 -> 90.8 mm
- net N$B13: track 0.00 -> 86.0 mm
- net N$C15: track 0.00 -> 73.9 mm
- net N$B11: track 0.00 -> 68.9 mm, vias 0 -> 1
- net N$B1: track 0.00 -> 68.0 mm, vias 0 -> 2
- net DGND: track 0.00 -> 65.6 mm
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Other:
- board size 255.2 x 103.8 mm -> 163.8 x 77.1 mm

Commit message: Add files via upload
Parts:
- moved R36 10.2 mm to (139.7, 49.5)
- moved R37 10.2 mm to (135.9, 49.5)
- moved R40 10.2 mm to (124.5, 49.5)
- moved R33 10.2 mm to (151.1, 49.5)
- moved R34 10.2 mm to (147.3, 49.5)
- moved R35 10.2 mm to (143.5, 49.5)
- moved R38 10.2 mm to (132.1, 49.5)
- moved R39 10.2 mm to (128.3, 49.5)
- moved SV11 10.2 mm to (133.3, 69.8)
- moved U5 10.2 mm to (137.2, 38.1)
- moved R25 7.62 mm to (120.7, 49.5)
- moved R27 7.62 mm to (113.0, 49.5)
- moved R28 7.62 mm to (109.2, 49.5)
- moved R29 7.62 mm to (105.4, 49.5)
- moved R30 7.62 mm to (101.6, 49.5)
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Connections:
- net AGND: no longer U6.4
- net VCC: now also U6.4
Routing:
- net AGND: track 556.8 -> 478.8 mm
- net VCC: track 356.2 -> 344.7 mm
- net N$10: track 167.1 -> 156.6 mm
- net N$48: track 167.5 -> 157.1 mm
- net N$47: track 175.7 -> 171.0 mm
- net N$1: track 37.6 -> 33.5 mm
- net N$C15: track 73.9 -> 78.0 mm
- net N$45: track 43.9 -> 40.1 mm
- net N$B12: track 90.8 -> 94.2 mm
- net N$C14: track 59.8 -> 62.6 mm
- net N$46: track 38.3 -> 35.8 mm
- net N$42: track 41.4 -> 38.8 mm
- net DGND: track 65.6 -> 63.1 mm
- net N$B13: track 86.0 -> 88.2 mm
- net N$64: track 8.94 -> 6.93 mm
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Other:
- board size 163.8 x 77.1 mm -> 153.7 x 77.1 mm
- board text added: "A10"
- board text added: "A11"
- board text added: "A8"
- board text added: "A9"

Commit message: Add files via upload
Parts:
- moved SV10 1.27 mm to (102.9, 68.6)
- moved SV11 1.27 mm to (133.3, 68.6)
- moved SV7 1.27 mm to (19.1, 68.6)
- moved SV8 1.27 mm to (41.9, 68.6)
- moved SV9 1.27 mm to (72.4, 68.6)
Routing:
- net N$10: track 156.6 -> 159.9 mm
- net N$5: track 36.8 -> 34.8 mm
- net N$7: track 32.7 -> 31.4 mm
- net N$21: track 34.8 -> 33.5 mm
- net N$9: track 37.3 -> 36.1 mm
- net N$8: track 34.0 -> 32.7 mm
- net N$6: track 31.4 -> 30.1 mm
- net N$49: track 37.5 -> 36.3 mm
- net N$41: track 36.3 -> 35.0 mm
- net N$40: track 35.0 -> 33.7 mm
- net N$4: track 38.1 -> 36.8 mm
- net N$39: track 34.8 -> 33.5 mm
- net N$30: track 35.8 -> 34.6 mm
- net N$28: track 35.0 -> 33.7 mm
- net N$27: track 36.3 -> 35.0 mm
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Other:
- outline, holes or cut-outs redrawn
- board text added: "5V"
- board text added: "A12"
- board text added: "A13"
- board text added: "A2"
- board text added: "B0"
- board text added: "B1"
- board text added: "B10"
- board text added: "B11"
- board text added: "B12"
- board text added: "B13"
- board text added: "B14"
- board text added: "B15"
- board text added: "B3"
- board text added: "B4"
- board text added: "B5"
- board text added: "B6"
- board text added: "B7"
- board text added: "B8"
- board text added: "B9"
- board text added: "C13"
- board text added: "C14"
- board text added: "C15"
- board text added: "GND"
- board text added: "IN"
- board text added: "VCC"
